File: OpenSourceDccDecoder/PCB/signal PCB/2-tone def.kicad_sch (KiCad schematic)
At the start: 5 parts, among them J11 Conn_01x04

Commit message: changed much of signal pcb tester
Parts:
- J11: footprint Connector_PinHeader_2.54mm:PinHeader_1x03_P2.54mm_Vertical -> custom_kicad_lib_sk:03_solderpad_2.54
Changed lines of the file:
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@@
       (effects (font (size 1.27 1.27)))
     )
-    (property "Footprint" "Connector_PinHeader_2.54mm:PinHeader_1x03_P2.54mm_Vertical" (at 86.614 54.61 0)
+    (property "Footprint" "custom_kicad_lib_sk:03_solderpad_2.54" (at 86.614 54.61 0)
       (effects (font (size 1.27 1.27)) hide)
     )
