File: OpenSourceDccDecoder/PCB/signal PCB/HV out.kicad_sch (KiCad schematic)
At the start: 11 parts, among them J1 Conn_01x06

Commit message: changed much of signal pcb tester
Parts:
- D1: footprint custom_kicad_lib_sk:LED_NO_SILK -> custom_kicad_lib_sk:02_solderpad_2.54
- J1: footprint Connector_PinHeader_2.54mm:PinHeader_1x06_P2.54mm_Vertical -> custom_kicad_lib_sk:06_solderpad_2.54
Changed lines of the file:
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@@
       (effects (font (size 1.27 1.27)))
     )
-    (property "Footprint" "Connector_PinHeader_2.54mm:PinHeader_1x06_P2.54mm_Vertical" (at 91.694 96.266 0)
+    (property "Footprint" "custom_kicad_lib_sk:06_solderpad_2.54" (at 91.694 96.266 0)
       (effects (font (size 1.27 1.27)) hide)
     )
@@
       (effects (font (size 1.27 1.27)) (justify right))
     )
-    (property "Footprint" "custom_kicad_lib_sk:LED_NO_SILK" (at 157.734 88.646 0)
+    (property "Footprint" "custom_kicad_lib_sk:02_solderpad_2.54" (at 157.734 88.646 0)
       (effects (font (size 1.27 1.27)) hide)
     )
