File: OpenSourceDccDecoder/PCB/signal PCB/UK-4tone w point.kicad_sch (KiCad schematic)
At the start: 11 parts, among them J1 Conn_01x06

Commit message: changed much of signal pcb tester
Parts:
- J1: footprint Connector_PinHeader_2.54mm:PinHeader_1x06_P2.54mm_Vertical -> custom_kicad_lib_sk:06_solderpad_2.54
Changed lines of the file:
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@@
       (effects (font (size 1.27 1.27)))
     )
-    (property "Footprint" "Connector_PinHeader_2.54mm:PinHeader_1x06_P2.54mm_Vertical" (at 85.09 80.01 0)
+    (property "Footprint" "custom_kicad_lib_sk:06_solderpad_2.54" (at 85.09 80.01 0)
       (effects (font (size 1.27 1.27)) hide)
     )

Commit message: added spread sheets for signal aspect images also swapped the LED connections in the Signal.cpp. They ordered in normal order from left to right
Parts:
- D1: footprint custom_kicad_lib_sk:LED_NO_SILK -> custom_kicad_lib_sk:02_solderpad_2.54
Changed lines of the file:
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@@
       (effects (font (size 1.27 1.27)) (justify right))
     )
-    (property "Footprint" "custom_kicad_lib_sk:LED_NO_SILK" (at 151.13 72.39 0)
+    (property "Footprint" "custom_kicad_lib_sk:02_solderpad_2.54" (at 151.13 72.39 0)
       (effects (font (size 1.27 1.27)) hide)
     )
