File: PCB/XnetBlockUnit/LDO.kicad_sch (KiCad schematic)
At the start: 4 parts, among them U401 L78L05_SOT89

Commit message: routed Xnet block unit. Ready for SMT assembly
Changed lines of the file:
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@@
-    (stroke (width 0) (type default))
-  )
-  (wire (pts (xy 177.8 87.63) (xy 177.8 88.9))
     (stroke (width 0) (type default))
   )
@@
     (effects (font (size 1.27 1.27)) (justify left))
   )
-  (symbol (lib_id "power:PWR_FLAG") (at 177.8 87.63 0) (unit 1)
-    (in_bom yes) (on_board yes) (dnp no) (fields_autoplaced)
-    (property "Reference" "#FLG0401" (at 177.8 85.725 0)
-      (effects (font (size 1.27 1.27)) hide)
-    )
-    (property "Value" "PWR_FLAG" (at 177.8 82.55 0)
-      (effects (font (size 1.27 1.27)))
-    )
-    (property "Footprint" "" (at 177.8 87.63 0)
-      (effects (font (size 1.27 1.27)) hide)
-    )
-    (property "Datasheet" "~" (at 177.8 87.63 0)
-      (effects (font (size 1.27 1.27)) hide)
-    )
-    (pin "1")
-    (instances
-      (project "XnetBlockUnit"
-        (path "/68824df7-235c-431f-a817-f5c5a64c6fe3/6de3bcf3-adb3-469c-8967-0d8d29e82b82"
-          (reference "#FLG0401") (unit 1)
-        )
-      )
-    )
-  )
   (symbol (lib_id "Device:C") (at 203.2 92.71 0) (unit 1)
