File: PCB/XnetBlockUnit/atmega.kicad_sch (KiCad schematic)
At the start: 9 parts, among them U201 HEADER_3x2, U202 ATmega328-A, Y201 Crystal_GND2

Commit message: routed Xnet block unit. Ready for SMT assembly
Changed lines of the file:
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@@
     (effects (font (size 1.27 1.27)) (justify left))
+  )
+  (hierarchical_label "GND" (shape passive) (at 162.56 127 270) (fields_autoplaced)
+    (effects (font (size 1.27 1.27)) (justify right))
   )
   (hierarchical_label "D2" (shape bidirectional) (at 186.69 101.6 0) (fields_autoplaced)
@@
         )
       )
-    )
-  )
-  (symbol (lib_id "power:GND") (at 162.56 127 0) (unit 1)
-    (in_bom yes) (on_board yes) (dnp no) (fields_autoplaced)
-    (property "Reference" "#PWR0202" (at 162.56 133.35 0)
-      (effects (font (size 1.27 1.27)) hide)
-    )
-    (property "Value" "GND" (at 162.56 131.4434 0)
-      (effects (font (size 1.27 1.27)))
-    )
-    (property "Footprint" "" (at 162.56 127 0)
-      (effects (font (size 1.27 1.27)) hide)
-    )
-    (property "Datasheet" "" (at 162.56 127 0)
-      (effects (font (size 1.27 1.27)) hide)
-    )
-    (pin "1")
-    (instances
-      (project "XnetBlockUnit"
-        (path "/68824df7-235c-431f-a817-f5c5a64c6fe3/5d46e491-9329-4a84-b412-faaf7812fe70"
-          (reference "#PWR0202") (unit 1)
-        )
-      )
-      (project "general_schematics"
-        (path "/e777d9ec-d073-4229-a9e6-2cf85636e407/f45deb4c-210f-430e-87b5-c6786dfa45a7"
-          (reference "#PWR054") (unit 1)
-        )
-      )

Commit message: many changes. Going to get some missing projects back
Changed lines of the file:
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@@
+    (effects (font (size 1.27 1.27)) (justify left))
+  )
+  (hierarchical_label "GND" (shape passive) (at 132.08 52.07 0) (fields_autoplaced)
     (effects (font (size 1.27 1.27)) (justify left))
   )
@@
         )
       )
-    )
-  )
-  (symbol (lib_id "power:GND") (at 132.08 52.07 0) (unit 1)
-    (in_bom yes) (on_board yes) (dnp no) (fields_autoplaced)
-    (property "Reference" "#PWR0201" (at 132.08 58.42 0)
-      (effects (font (size 1.27 1.27)) hide)
-    )
-    (property "Value" "GND" (at 132.08 56.5134 0)
-      (effects (font (size 1.27 1.27)))
-    )
-    (property "Footprint" "" (at 132.08 52.07 0)
-      (effects (font (size 1.27 1.27)) hide)
-    )
-    (property "Datasheet" "" (at 132.08 52.07 0)
-      (effects (font (size 1.27 1.27)) hide)
-    )
-    (pin "1")
-    (instances
-      (project "XnetBlockUnit"
-        (path "/68824df7-235c-431f-a817-f5c5a64c6fe3/5d46e491-9329-4a84-b412-faaf7812fe70"
-          (reference "#PWR0201") (unit 1)
-        )
-      )
-      (project "general_schematics"
-        (path "/e777d9ec-d073-4229-a9e6-2cf85636e407/f45deb4c-210f-430e-87b5-c6786dfa45a7"
-          (reference "#PWR053") (unit 1)
-        )
-      )
