File: PCB/XnetBlockUnit/XnetBlockUnit.kicad_pcb (KiCad board)
At the start: 2 copper layers, 51.5 x 74 mm, 53 parts, among them J101 sensor, J102 Screw_Terminal_01x08, J103 Screw_Terminal_01x08, J301 RJ12, J302 RJ12, U201 HEADER_3x2, U202 ATmega328-A, U301 MAX485E, U401 L78L05_SOT89, U501 EL814, U601 EL814, Y201 Crystal_GND2

Commit message: routed Xnet block unit. Ready for SMT assembly
Parts:
- added G***: LOGO, custom_kicad_lib_sk:Train-Science logo small, F.Cu at (63.2, 110.6)
- added R102: 1k, custom_kicad_lib_sk:R_0603_smalltext, F.Cu at (58.0, 113.5)
- R101: value 1k -> 100R
- moved R101 21.9 mm to (76.3, 128.1)
- moved U201 5.04 mm to (41.8, 77.7)
- moved R201 5.02 mm to (67.8, 97.0), turned to -90 degrees
- moved D201 3.18 mm to (67.8, 101.1), turned to 90 degrees
- moved C101 2.16 mm to (75.1, 133.6), turned to 180 degrees
- moved R202 1.00 mm to (47.5, 81.6)
Connections:
- net /Mosfet/Coil_A_TTL renamed /coil_A_TTL
- net /Mosfet/Coil_B_TTL renamed /coil_B_TTL
- D101 pad 3: /coil_pow -> Net-(D101-+)
- R101 pad 1: +5V -> /coil_pow
- R101 pad 2: Net-(JP101-B) -> Net-(D101-+)
- R801 pad 1: /atmega/D6 -> /signal_R
- R802 pad 1: /atmega/D5 -> /signal_g
- U202 pad 10: /atmega/D6 -> /sens_1
- U202 pad 13: /atmega/D9 -> /signal_g
- U202 pad 14: /atmega/D10 -> /signal_R
- U202 pad 9: /atmega/D5 -> /sens_2
- U501 pad 4: /atmega/D3 -> /sens_1
- U601 pad 4: /atmega/D4 -> /sens_2
Routing:
- net +5V: track 11.0 -> 90.5 mm, vias 0 -> 6
- net +12V: track 1.99 -> 60.0 mm, vias 0 -> 1
- net /atmega/LED: track 0.00 -> 44.1 mm, vias 0 -> 4
- net /coil_pow: track 0.00 -> 43.5 mm
- net /atmega/MOSI: track 0.00 -> 41.4 mm, vias 0 -> 2
- net /atmega/MISO: track 0.00 -> 41.4 mm, vias 0 -> 2
- net /sensor1/TRACK: track 0.00 -> 36.2 mm
- net /Out: track 0.00 -> 32.6 mm
- net /Xnet/A: track 0.00 -> 28.8 mm
- net /atmega/reset: track 0.00 -> 28.6 mm, vias 0 -> 4
- net /Xnet/B: track 0.00 -> 25.2 mm
- net /signal_R: track 0.00 -> 24.6 mm
- net /sens_2: track 0.00 -> 22.6 mm
- net /sensor1/COM: track 3.70 -> 23.5 mm
- net /sens_1: track 0.00 -> 17.4 mm
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- added copper zone on B.Cu, net GND
- added copper zone on F.Cu, net GND
Other:
- board text added: "ADD"
- board text added: "AUTO"
- board text added: "COM"
- board text added: "GND"
- board text added: "GO"
- board text added: "ICSP"
- board text added: "In"
- board text added: "OUT"
- board text added: "SYNCH"
- board text added: "Xnet"
- board text added: "Xnet block module"
- board text added: "coil +"
- board text added: "coil A"
- board text added: "green"
- board text added: "power AC/DC"
- board text added: "red"
- board text added: "sensor1"
- board text added: "sensor2"
- board text added: "signal +"

Commit message: many changes. Going to get some missing projects back
Parts:
- added C102: 100nF, Capacitor_SMD:C_0603_1608Metric_Pad1.08x0.95mm_HandSolder, F.Cu at (84.6, 83.2)
- added RV101: R_Potentiometer, Potentiometer_THT:Potentiometer_Runtron_RM-065_Vertical, F.Cu at (83.7, 80.9)
Routing:
- net /atmega/A6: track 0.00 -> 40.3 mm, vias 0 -> 4
- net +5V: track 90.5 -> 130.6 mm
- net GND: vias 117 -> 120

Commit message: added some files
Other:
- board text added: "+"
- board text added: "-"
- board text added: "~"
Changed lines of the file:
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@@
+    (effects (font (size 0.5 0.5) (thickness 0.075)) (justify left bottom))
+  )
+  (gr_text "~" (at 86.36 131.064) (layer "F.SilkS")
     (effects (font (size 0.5 0.5) (thickness 0.075)) (justify left bottom))
   )
@@
     (effects (font (size 0.5 0.5) (thickness 0.075)) (justify left bottom))
   )
+  (gr_text "-" (at 77.978 131.953) (layer "F.SilkS")
+    (effects (font (size 0.5 0.5) (thickness 0.075)) (justify left bottom))
+  )
   (gr_text "COM" (at 57.658 138.938) (layer "F.SilkS")
     (effects (font (size 0.5 0.5) (thickness 0.075)) (justify left bottom))
@@
     (effects (font (size 0.5 0.5) (thickness 0.075)) (justify left bottom))
   )
+  (gr_text "+" (at 78.486 126.873) (layer "F.SilkS")
+    (effects (font (size 0.5 0.5) (thickness 0.075)) (justify left bottom))
+  )
+  (gr_text "~" (at 86.487 128.397) (layer "F.SilkS")
+    (effects (font (size 0.5 0.5) (thickness 0.075)) (justify left bottom))
+  )
