File: PCB/XnetBlockUnit/XnetBlockUnit.kicad_sch (KiCad schematic)
At the start: 7 parts, among them J101 sensor, J102 Screw_Terminal_01x08, J103 Screw_Terminal_01x08

Commit message: routed Xnet block unit. Ready for SMT assembly
Parts:
- added R101: 100R, custom_kicad_lib_sk:R_0603_smalltext, symbol resistors_0603:R_100R_0603
- renumbered R101 to R102
Connections:
- net coil_pow: now also R101.1; no longer D?.3 (+)
- new net: D?.3 (+), R101.2
- no-connect marks 0 -> 6
Other:
- moved on the sheet: C101

Commit message: many changes. Going to get some missing projects back
Parts:
- added C202: 100nF, Capacitor_SMD:C_0603_1608Metric_Pad1.08x0.95mm_HandSolder, symbol Device:C
- added RV101: R_Potentiometer, Potentiometer_THT:Potentiometer_Runtron_RM-065_Vertical, symbol Device:R_Potentiometer
Connections:
- net +5V: now also RV101.3
- net GND: now also C202.1, RV101.1
- net atmega/A6: now also C202.2, RV101.2
- no-connect marks 6 -> 5
Changed lines of the file:
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@@
 (kicad_sch (version 20230121) (generator eeschema)
   (paper "A4")
+  (junction (at 86.36 119.38) (diameter 0) (color 0 0 0 0)
+  )
   (junction (at 124.46 55.88) (diameter 0) (color 0 0 0 0)
   )
@@
   (no_connect (at 76.2 102.87))
   (no_connect (at 78.74 80.01))
-  (no_connect (at 76.2 100.33))
   (wire (pts (xy 115.57 135.89) (xy 115.57 138.43))
     (stroke (width 0) (type default))
@@
     (stroke (width 0) (type default))
   )
+  (wire (pts (xy 86.36 100.33) (xy 76.2 100.33))
+    (stroke (width 0) (type default))
+  )
   (wire (pts (xy 116.84 55.88) (xy 124.46 55.88))
     (stroke (width 0) (type default))
@@
     (stroke (width 0) (type default))
   )
+  (wire (pts (xy 93.98 114.3) (xy 93.98 115.57))
+    (stroke (width 0) (type default))
+  )
   (wire (pts (xy 133.35 104.14) (xy 163.83 104.14))
     (stroke (width 0) (type default))
@@
     (stroke (width 0) (type default))
   )
+  (wire (pts (xy 86.36 119.38) (xy 86.36 100.33))
+    (stroke (width 0) (type default))
+  )
   (wire (pts (xy 140.97 93.98) (xy 140.97 83.82))
     (stroke (width 0) (type default))
@@
     (stroke (width 0) (type default))
   )
+  (wire (pts (xy 86.36 127) (xy 86.36 128.27))
+    (stroke (width 0) (type default))
+  )
   (wire (pts (xy 80.01 87.63) (xy 76.2 87.63))
     (stroke (width 0) (type default))
@@
     (stroke (width 0) (type default))
   )
+  (wire (pts (xy 86.36 119.38) (xy 90.17 119.38))
+    (stroke (width 0) (type default))
+  )
   (wire (pts (xy 124.46 54.61) (xy 124.46 55.88))
     (stroke (width 0) (type default))
@@
   )
   (wire (pts (xy 124.46 45.72) (xy 124.46 46.99))
+    (stroke (width 0) (type default))
+  )
+  (wire (pts (xy 93.98 123.19) (xy 93.98 128.27))
     (stroke (width 0) (type default))
   )
@@
   (label "coil_B" (at 125.73 99.06 0) (fields_autoplaced)
     (effects (font (size 1.27 1.27)) (justify left bottom))
+  )
+  (symbol (lib_id "Device:C") (at 86.36 123.19 180) (unit 1)
+    (in_bom yes) (on_board yes) (dnp no)
+    (property "Reference" "C202" (at 78.74 121.92 0)
+      (effects (font (size 1.27 1.27)) (justify right))
+    )
+    (property "Value" "100nF" (at 77.47 124.46 0)
+      (effects (font (size 1.27 1.27)) (justify right))
+    )
+    (property "Footprint" "Capacitor_SMD:C_0603_1608Metric_Pad1.08x0.95mm_HandSolder" (at 85.3948 119.38 0)
+      (effects (font (size 1.27 1.27)) hide)
+    )
+    (property "Datasheet" "~" (at 86.36 123.19 0)
+      (effects (font (size 1.27 1.27)) hide)
+    )
+    (property "JLCPCB Part#" "C14663" (at 86.36 123.19 0)
+      (effects (font (size 1.27 1.27)) hide)
+    )
+    (pin "1")
+    (pin "2")
+    (instances
+      (project "XnetBlockUnit"
+        (path "/68824df7-235c-431f-a817-f5c5a64c6fe3/5d46e491-9329-4a84-b412-faaf7812fe70"
+          (reference "C202") (unit 1)
+        )
+        (path "/68824df7-235c-431f-a817-f5c5a64c6fe3"
+          (reference "C102") (unit 1)
+        )
+      )
+      (project "general_schematics"
+        (path "/e777d9ec-d073-4229-a9e6-2cf85636e407/f45deb4c-210f-430e-87b5-c6786dfa45a7"
+          (reference "C13") (unit 1)
+        )
+      )
+    )
+  )
+  (symbol (lib_id "power:GND") (at 86.36 128.27 0) (unit 1)
+    (in_bom yes) (on_board yes) (dnp no) (fields_autoplaced)
+    (property "Reference" "#PWR0118" (at 86.36 134.62 0)
+      (effects (font (size 1.27 1.27)) hide)
+    )
+    (property "Value" "GND" (at 86.36 132.215 0)
+      (effects (font (size 1.27 1.27)))
+    )
+    (property "Footprint" "" (at 86.36 128.27 0)
+      (effects (font (size 1.27 1.27)) hide)
+    )
+    (property "Datasheet" "" (at 86.36 128.27 0)
+      (effects (font (size 1.27 1.27)) hide)
+    )
+    (pin "1")
+    (instances
+      (project "XnetBlockUnit"
+        (path "/68824df7-235c-431f-a817-f5c5a64c6fe3"
+          (reference "#PWR0118") (unit 1)
+        )
+      )
+    )
   )
   (symbol (lib_id "Diode_Bridge:MB6S") (at 132.08 124.46 180) (unit 1)
@@
         (path "/68824df7-235c-431f-a817-f5c5a64c6fe3"
           (reference "JP101") (unit 1)
+        )
+      )
+    )
+  )
+  (symbol (lib_id "power:GND") (at 93.98 128.27 0) (unit 1)
+    (in_bom yes) (on_board yes) (dnp no) (fields_autoplaced)
+    (property "Reference" "#PWR0116" (at 93.98 134.62 0)
+      (effects (font (size 1.27 1.27)) hide)
+    )
+    (property "Value" "GND" (at 93.98 132.215 0)
+      (effects (font (size 1.27 1.27)))
+    )
+    (property "Footprint" "" (at 93.98 128.27 0)
+      (effects (font (size 1.27 1.27)) hide)
+    )
+    (property "Datasheet" "" (at 93.98 128.27 0)
+      (effects (font (size 1.27 1.27)) hide)
+    )
+    (pin "1")
+    (instances
+      (project "XnetBlockUnit"
+        (path "/68824df7-235c-431f-a817-f5c5a64c6fe3"
+          (reference "#PWR0116") (unit 1)
         )
       )
@@
     )
   )
+  (symbol (lib_id "Device:R_Potentiometer") (at 93.98 119.38 180) (unit 1)
+    (in_bom yes) (on_board yes) (dnp no) (fields_autoplaced)
+    (property "Reference" "RV101" (at 95.758 118.356 0)
+      (effects (font (size 1.27 1.27)) (justify right))
+    )
+    (property "Value" "R_Potentiometer" (at 95.758 120.404 0)
+      (effects (font (size 1.27 1.27)) (justify right))
+    )
+    (property "Footprint" "Potentiometer_THT:Potentiometer_Runtron_RM-065_Vertical" (at 93.98 119.38 0)
+      (effects (font (size 1.27 1.27)) hide)
+    )
+    (property "Datasheet" "~" (at 93.98 119.38 0)
+      (effects (font (size 1.27 1.27)) hide)
+    )
+    (pin "1")
+    (pin "2")
+    (pin "3")
+    (instances
+      (project "XnetBlockUnit"
+        (path "/68824df7-235c-431f-a817-f5c5a64c6fe3"
+          (reference "RV101") (unit 1)
+        )
+      )
+    )
+  )
   (symbol (lib_id "Device:C_Polarized") (at 115.57 132.08 0) (unit 1)
     (in_bom yes) (on_board yes) (dnp no)
@@
         )
       )
+    )
+  )
+  (symbol (lib_id "power:+5V") (at 93.98 114.3 0) (unit 1)
+    (in_bom yes) (on_board yes) (dnp no) (fields_autoplaced)
+    (property "Reference" "#PWR0117" (at 93.98 118.11 0)
+      (effects (font (size 1.27 1.27)) hide)
+    )
+    (property "Value" "+5V" (at 93.98 110.355 0)
+      (effects (font (size 1.27 1.27)))
+    )
+    (property "Footprint" "" (at 93.98 114.3 0)
+      (effects (font (size 1.27 1.27)) hide)
+    )
+    (property "Datasheet" "" (at 93.98 114.3 0)
+      (effects (font (size 1.27 1.27)) hide)
+    )
+    (pin "1")
+    (instances
+      (project "XnetBlockUnit"
+        (path "/68824df7-235c-431f-a817-f5c5a64c6fe3"
+          (reference "#PWR0117") (unit 1)
+        )
+      )

Commit message: added some files
Parts:
- gave numbers to parts that had none: 1
- renumbered C202 to C102
Changed lines of the file:
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@@
   (symbol (lib_id "Device:C") (at 86.36 123.19 180) (unit 1)
     (in_bom yes) (on_board yes) (dnp no)
-    (property "Reference" "C202" (at 78.74 121.92 0)
+    (property "Reference" "C102" (at 78.74 121.92 0)
       (effects (font (size 1.27 1.27)) (justify right))
     )
@@
     (instances
       (project "XnetBlockUnit"
-        (path "/68824df7-235c-431f-a817-f5c5a64c6fe3/5d46e491-9329-4a84-b412-faaf7812fe70"
-          (reference "C202") (unit 1)
-        )
         (path "/68824df7-235c-431f-a817-f5c5a64c6fe3"
           (reference "C102") (unit 1)
@@
   (symbol (lib_id "Diode_Bridge:MB6S") (at 132.08 124.46 180) (unit 1)
     (in_bom yes) (on_board yes) (dnp no)
-    (property "Reference" "D?" (at 127 128.27 0)
+    (property "Reference" "D101" (at 127 128.27 0)
       (effects (font (size 1.27 1.27)))
     )
@@
     (instances
       (project "XnetBlockUnit"
-        (path "/68824df7-235c-431f-a817-f5c5a64c6fe3/e7736df0-222d-4298-ac34-425fe37226f4"
-          (reference "D?") (unit 1)
-        )
-        (path "/68824df7-235c-431f-a817-f5c5a64c6fe3/ed123d09-0416-4e37-84e2-70dd62f130a4"
-          (reference "D?") (unit 1)
-        )
         (path "/68824df7-235c-431f-a817-f5c5a64c6fe3"
           (reference "D101") (unit 1)
