File: PCB/DCC_NANO_SHIELD/DCC_NANO_SHIELD.kicad_sch (KiCad schematic)
At the start: 14 parts, among them J1 Screw_Terminal_01x02, SW1 config, U1 6N137, U2 Buck

Commit message: many changes. Going to get some missing projects back
Parts:
- D11: value (none) -> D; footprint (none) -> Diode_SMD:D_1206_3216Metric_Pad1.42x1.75mm_HandSolder
- R11: value (none) -> 1k; footprint (none) -> Resistor_SMD:R_0805_2012Metric_Pad1.20x1.40mm_HandSolder
- R21, R31: value (none) -> 10k; footprint (none) -> Resistor_SMD:R_0805_2012Metric_Pad1.20x1.40mm_HandSolder
