File: OS-ServoDriver/DCC.kicad_sch (KiCad schematic)
At the start: 5 parts, among them U701 6N137

Commit message: added schematics to incorporate company name
Other:
- company: (none) -> Train-Science
Changed lines of the file:
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@@
 (kicad_sch (version 20230121) (generator eeschema)
   (paper "A4")
+  (title_block
+    (company "Train-Science")
+  )
   (junction (at 151.13 96.52) (diameter 0) (color 0 0 0 0)
   )

Commit message: commit 4 push
Parts:
- removed D701: 1N4148WS, Diode_SMD:D_SOD-323, symbol custom_kicad_lib_sk:1N4148WS
- removed R701: 1k5, custom_kicad_lib_sk:R_0603_smalltext, symbol resistors_0603:R_1k5_0603
- removed R702, R703: 10k, custom_kicad_lib_sk:R_0603_smalltext, symbol resistors_0603:R_10k_0603
- added D1001: 1N4148WS, Diode_SMD:D_SOD-323, symbol custom_kicad_lib_sk:1N4148WS
- added R1001: 1k, custom_kicad_lib_sk:R_0603_smalltext, symbol resistors_0603:R_1k_0603
- added R1002, R1003: 10k, custom_kicad_lib_sk:R_0603_smalltext, symbol resistors_0603:R_10k_0603
- renumbered U701 to U1001
Connections:
- net 5V: now also R1002.1, R1003.1
- net DCC_A: now also R1001.1
- net DCC_B: now also D1001.2 (A)
- net DCC_TTL: now also R1003.2
- net at U1001.7 (EN): now also R1002.2
- net at U1001.2 (A): now also D1001.1 (K), R1001.2
Other:
- company: Train-Science -> (none)
