File: OS-ServoDriver/buck.kicad_sch (KiCad schematic)
At the start: 11 parts, among them U901 MT2499A

Commit message: added schematics to incorporate company name
Other:
- company: (none) -> Train-Science
Changed lines of the file:
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@@
 (kicad_sch (version 20230121) (generator eeschema)
   (paper "A4")
+  (title_block
+    (company "Train-Science")
+  )
   (junction (at 101.6 74.93) (diameter 0) (color 0 0 0 0)
   )

Commit message: commit 4 push
Connections:
- net Vin renamed VDC_in
Other:
- company: Train-Science -> (none)
Changed lines of the file:
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@@
 (kicad_sch (version 20230121) (generator eeschema)
   (paper "A4")
-  (title_block
-    (company "Train-Science")
-  )
   (junction (at 101.6 74.93) (diameter 0) (color 0 0 0 0)
   )
@@
     (effects (font (size 1.27 1.27)) (justify left))
   )
-  (hierarchical_label "Vin" (shape passive) (at 101.6 72.39 180) (fields_autoplaced)
+  (hierarchical_label "VDC_in" (shape passive) (at 101.6 72.39 180) (fields_autoplaced)
     (effects (font (size 1.27 1.27)) (justify right))
   )
@@
     (pin "2")
     (instances
-      (project "OS-ServoDriver"
-        (path "/6c2c208c-97cf-495d-b492-7f3fa6958cdd/09fa05e0-8432-45ce-9107-75e3f3cdb40f"
+      (project "OS-servoDriver"
+        (path "/b6ccf16f-5cc5-4d5a-97fc-20f76ee5c73e/7745b34c-3ce1-4fee-9e05-e2cc7dc8f5e5"
           (reference "R903") (unit 1)
         )
@@
     (pin "2")
     (instances
-      (project "OS-ServoDriver"
-        (path "/6c2c208c-97cf-495d-b492-7f3fa6958cdd/09fa05e0-8432-45ce-9107-75e3f3cdb40f"
+      (project "OS-servoDriver"
+        (path "/b6ccf16f-5cc5-4d5a-97fc-20f76ee5c73e/7745b34c-3ce1-4fee-9e05-e2cc7dc8f5e5"
           (reference "C902") (unit 1)
         )
@@
     (pin "2")
     (instances
-      (project "OS-ServoDriver"
-        (path "/6c2c208c-97cf-495d-b492-7f3fa6958cdd/09fa05e0-8432-45ce-9107-75e3f3cdb40f"
+      (project "OS-servoDriver"
+        (path "/b6ccf16f-5cc5-4d5a-97fc-20f76ee5c73e/7745b34c-3ce1-4fee-9e05-e2cc7dc8f5e5"
           (reference "C903") (unit 1)
         )
@@
     (pin "2")
     (instances
-      (project "OS-ServoDriver"
-        (path "/6c2c208c-97cf-495d-b492-7f3fa6958cdd/09fa05e0-8432-45ce-9107-75e3f3cdb40f"
+      (project "OS-servoDriver"
+        (path "/b6ccf16f-5cc5-4d5a-97fc-20f76ee5c73e/7745b34c-3ce1-4fee-9e05-e2cc7dc8f5e5"
           (reference "L901") (unit 1)
         )
@@
     (pin "2")
     (instances
-      (project "OS-ServoDriver"
-        (path "/6c2c208c-97cf-495d-b492-7f3fa6958cdd/09fa05e0-8432-45ce-9107-75e3f3cdb40f"
+      (project "OS-servoDriver"
+        (path "/b6ccf16f-5cc5-4d5a-97fc-20f76ee5c73e/7745b34c-3ce1-4fee-9e05-e2cc7dc8f5e5"
           (reference "C905") (unit 1)
         )
@@
     (pin "2")
     (instances
-      (project "OS-ServoDriver"
-        (path "/6c2c208c-97cf-495d-b492-7f3fa6958cdd/09fa05e0-8432-45ce-9107-75e3f3cdb40f"
+      (project "OS-servoDriver"
+        (path "/b6ccf16f-5cc5-4d5a-97fc-20f76ee5c73e/7745b34c-3ce1-4fee-9e05-e2cc7dc8f5e5"
           (reference "C901") (unit 1)
         )
@@
     (pin "2")
     (instances
-      (project "OS-ServoDriver"
-        (path "/6c2c208c-97cf-495d-b492-7f3fa6958cdd/09fa05e0-8432-45ce-9107-75e3f3cdb40f"
+      (project "OS-servoDriver"
+        (path "/b6ccf16f-5cc5-4d5a-97fc-20f76ee5c73e/7745b34c-3ce1-4fee-9e05-e2cc7dc8f5e5"
           (reference "R902") (unit 1)
         )
@@
     (pin "9")
     (instances
-      (project "OS-ServoDriver"
-        (path "/6c2c208c-97cf-495d-b492-7f3fa6958cdd/09fa05e0-8432-45ce-9107-75e3f3cdb40f"
+      (project "OS-servoDriver"
+        (path "/b6ccf16f-5cc5-4d5a-97fc-20f76ee5c73e/7745b34c-3ce1-4fee-9e05-e2cc7dc8f5e5"
           (reference "U901") (unit 1)
         )
@@
     (pin "2")
     (instances
-      (project "OS-ServoDriver"
-        (path "/6c2c208c-97cf-495d-b492-7f3fa6958cdd/09fa05e0-8432-45ce-9107-75e3f3cdb40f"
+      (project "OS-servoDriver"
+        (path "/b6ccf16f-5cc5-4d5a-97fc-20f76ee5c73e/7745b34c-3ce1-4fee-9e05-e2cc7dc8f5e5"
           (reference "C904") (unit 1)
         )
@@
     (pin "2")
     (instances
-      (project "OS-ServoDriver"
-        (path "/6c2c208c-97cf-495d-b492-7f3fa6958cdd/09fa05e0-8432-45ce-9107-75e3f3cdb40f"
+      (project "OS-servoDriver"
+        (path "/b6ccf16f-5cc5-4d5a-97fc-20f76ee5c73e/7745b34c-3ce1-4fee-9e05-e2cc7dc8f5e5"
           (reference "R901") (unit 1)
         )
@@
     )
   )
+  (symbol (lib_id "power:PWR_FLAG") (at 176.53 74.93 0) (unit 1)
+    (in_bom yes) (on_board yes) (dnp no) (fields_autoplaced)
+    (property "Reference" "#FLG01101" (at 176.53 73.025 0)
+      (effects (font (size 1.27 1.27)) hide)
+    )
+    (property "Value" "PWR_FLAG" (at 176.53 69.85 0)
+      (effects (font (size 1.27 1.27)))
+    )
+    (property "Footprint" "" (at 176.53 74.93 0)
+      (effects (font (size 1.27 1.27)) hide)
+    )
+    (property "Datasheet" "~" (at 176.53 74.93 0)
+      (effects (font (size 1.27 1.27)) hide)
+    )
+    (pin "1")
+    (instances
+      (project "OS-servoDriver"
+        (path "/b6ccf16f-5cc5-4d5a-97fc-20f76ee5c73e/0c27c8b7-3734-4129-8cd0-d3d033ef2608"
+          (reference "#FLG01101") (unit 1)
+        )
+        (path "/b6ccf16f-5cc5-4d5a-97fc-20f76ee5c73e/7745b34c-3ce1-4fee-9e05-e2cc7dc8f5e5"
+          (reference "#FLG0501") (unit 1)
+        )
+      )
+    )
+  )
   (symbol (lib_id "Device:C") (at 186.69 85.09 0) (unit 1)
     (in_bom yes) (on_board yes) (dnp no) (fields_autoplaced)
@@
     (pin "2")
     (instances
-      (project "OS-ServoDriver"
-        (path "/6c2c208c-97cf-495d-b492-7f3fa6958cdd/09fa05e0-8432-45ce-9107-75e3f3cdb40f"
+      (project "OS-servoDriver"
+        (path "/b6ccf16f-5cc5-4d5a-97fc-20f76ee5c73e/7745b34c-3ce1-4fee-9e05-e2cc7dc8f5e5"
           (reference "C906") (unit 1)
         )

Commit message: Changed OSSD code to retain aspects in EEPROM. In the event that the power has been cut-off. The OSSD can resume it's last known state. This is untested and I may want to change this into an option.
Parts:
- C903: JLCPCB Part# C1729 -> C1532
- L901: JLCPCB Part# C2929438 -> C92945
Changed lines of the file:
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@@
       (effects (font (size 1.27 1.27)) hide)
     )
-    (property "JLCPCB Part#" "C1729" (at 139.7 63.5 90)
+    (property "JLCPCB Part#" "C1532" (at 139.7 63.5 90)
       (effects (font (size 1.27 1.27)) hide)
     )
@@
       (effects (font (size 1.27 1.27)) hide)
     )
-    (property "JLCPCB Part#" "C2929438" (at 149.86 74.93 90)
+    (property "JLCPCB Part#" "C92945" (at 149.86 74.93 90)
       (effects (font (size 1.27 1.27)) hide)
     )
