File: OS-S88n/OS-S88n.kicad_sch (KiCad schematic)
At the start: 2 parts, among them J103 Screw_Terminal_01x09, J104 Screw_Terminal_01x09

Commit message: added missing S88 files to repo
Parts:
- removed J103, J104: Screw_Terminal_01x09, TerminalBlock_Phoenix:TerminalBlock_Phoenix_MKDS-1,5-9-5.08_1x09_P5.08mm_Horizontal, symbol Connector:Screw_Terminal_01x09
- added J? (x6): Screw_Terminal_01x03, symbol Connector:Screw_Terminal_01x03
Connections:
- net COM: now also J?.1 (Pin_1), J?.3 (Pin_3)
- net CS1/TRACK: now also J?.1 (Pin_1)
- net CS10/TRACK: now also J?.3 (Pin_3)
- net CS11/TRACK: now also J?.1 (Pin_1)
- net CS12/TRACK: now also J?.2 (Pin_2)
- net CS13/TRACK: now also J?.3 (Pin_3)
- net CS14/TRACK: now also J?.1 (Pin_1)
- net CS15/TRACK: now also J?.2 (Pin_2)
- net CS16/TRACK: now also J?.3 (Pin_3)
- net CS2/TRACK: now also J?.2 (Pin_2)
- net CS3/TRACK: now also J?.3 (Pin_3)
- net CS4/TRACK: now also J?.1 (Pin_1)
- net CS5/TRACK: now also J?.2 (Pin_2)
- net CS6/TRACK: now also J?.3 (Pin_3)
- net CS7/TRACK: now also J?.1 (Pin_1)
- net CS8/TRACK: now also J?.2 (Pin_2)
- net CS9/TRACK: now also J?.2 (Pin_2)
