File: OS-S88n/RJ45.kicad_sch (KiCad schematic)
At the start: 2 parts, among them J2101 RJ45, J2102 RJ45

Commit message: added missing S88 files to repo
Parts:
- added Q?: BC847, Package_TO_SOT_SMD:SOT-23, symbol custom_kicad_lib_sk:BC847
- added R?: 100k, custom_kicad_lib_sk:R_0603_smalltext, symbol resistors_0603:R_100k_0603
- added R?: 4k7, custom_kicad_lib_sk:R_0603_smalltext, symbol resistors_0603:R_4k7_0603
- J2101, J2102: JLCPCB Part# (none) -> C2847314
Connections:
- net CLOCK: now also J2102.4; no longer J2102.5
- net DATA_OUT: now also J2102.2; no longer J2102.7
- net GND: now also J2102.3, J2102.5, Q?.2 (E); no longer J2102.4, J2102.6
- net PL: now also J2102.6; no longer J2102.3
- net RESET: now also Q?.3 (C), R?.2; no longer J2101.7, J2102.2
- net VCC: now also J2102.1, R?.1; no longer J2102.8
- new net: J2101.7, J2102.7, R?.1
- new net: Q?.1 (B), R?.2
- no-connect marks 0 -> 2
