File: OS-S88n/SR latch.kicad_sch (KiCad schematic)
At the start: 7 parts, among them Q301 BC847

Commit message: added missing S88 files to repo
Parts:
- removed Q301: BC847, Package_TO_SOT_SMD:SOT-23, symbol custom_kicad_lib_sk:BC847
- removed R301: 4k7, custom_kicad_lib_sk:R_0603_smalltext, symbol resistors_0603:R_4k7_0603
- removed R302: 100k, custom_kicad_lib_sk:R_0603_smalltext, symbol resistors_0603:R_100k_0603
Connections:
- net RESET: now also U?.12 (R3), U?.12 (R3), U?.14 (R4), U?.14 (R4), U?.4 (R1), U?.4 (R1), U?.6 (R2), U?.6 (R2)
