File: PCB/analog_solutions/CDU/CDU.kicad_pcb (KiCad board)
At the start: 2 copper layers, 38 x 37 mm, 18 parts, among them J1001 Screw_Terminal_01x02, J1002 Screw_Terminal_01x02, Q1001 4A_DARLINGTON

Commit message: many changes
Other:
- board text added: "+"
Changed lines of the file:
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@@
+    (effects (font (size 0.5 0.5) (thickness 0.075)) (justify left bottom))
+  )
+  (gr_text "+" (at 113.5 60) (layer "F.SilkS")
     (effects (font (size 0.5 0.5) (thickness 0.075)) (justify left bottom))
   )
