File: PCB/blockModules/digital/BloX ABC MkII/CS.kicad_sch (KiCad schematic)
At the start: 6 parts, among them U302 EL814

Commit message: added some files
Parts:
- removed D301, D302, D303, D304: SS53, Diode_SMD:D_SMA, symbol custom_kicad_lib_sk:SS53
- added D401: D_Bridge_+-AA, custom_kicad_lib_sk:DB201S, symbol Device:D_Bridge_+-AA
Connections:
- net COM: now also D401.4
- net TRACK: now also D401.3
- new net: D401.1 (+), D401.2 (-)
Other:
- moved on the sheet: R301, U302
