File: PCB/DECODERS_N_OCCUPANCY/OSSD/src/PCB/OSSD/mosfets.kicad_sch (KiCad schematic)
At the start: 9 parts

Commit message: Added PDF files for all schematics
Parts:
- J11: footprint TerminalBlock_Phoenix:TerminalBlock_Phoenix_MKDS-1,5-3-5.08_1x03_P5.08mm_Horizontal -> Connector_Phoenix_MC:PhoenixContact_MC_1,5_3-G-3.5_1x03_P3.50mm_Horizontal; JLCPCB Part# (none) -> C430551
Changed lines of the file:
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@@
 			)
 		)
-		(property "Footprint" "TerminalBlock_Phoenix:TerminalBlock_Phoenix_MKDS-1,5-3-5.08_1x03_P5.08mm_Horizontal"
+		(property "Footprint" "Connector_Phoenix_MC:PhoenixContact_MC_1,5_3-G-3.5_1x03_P3.50mm_Horizontal"
 			(at 166.37 34.29 0)
 			(effects
@@
 			(at 166.37 34.29 0)
 			(effects
+				(font
+					(size 1.27 1.27)
+				)
+				(hide yes)
+			)
+		)
+		(property "JLCPCB Part#" "C430551"
+			(at 166.37 34.29 0)
+			(effects
