File: PCB_SOURCE/Academy/ledStripSchematic/ledStrip.kicad_pcb (KiCad board)
At the start: 2 copper layers, 243 x 27 mm, 47 parts, among them J1 Conn_01x01_Pin, J2 Conn_01x01_Pin, J3 Conn_01x01_Pin, J4 Conn_01x01_Pin, U1 LM317_TO-252

Commit message: added some files, but mainly this is to update hex file of OSSD
Parts:
- removed ?: , 
- moved REF** 1.00 mm to (38.0, 110.2)
- moved REF** 1.00 mm to (245.2, 125.2)
- moved REF** 1.00 mm to (37.8, 124.2)
- moved REF** 1.00 mm to (245.5, 111.2)
- moved D9 0.57 mm to (66.0, 130.4)
- moved R4 0.57 mm to (56.4, 130.4)
- moved D12 0.50 mm to (108.5, 130.5)
- moved D16 0.50 mm to (153.5, 130.5)
- moved D19 0.50 mm to (198.5, 130.5)
- moved D22 0.50 mm to (243.5, 130.5)
- moved R5 0.50 mm to (112.5, 130.5)
Routing:
- net AC2: track 252.2 -> 250.2 mm
- net AC1: track 256.6 -> 255.7 mm
- net /Vled: track 234.3 -> 233.7 mm, vias 4 -> 8
- net Net-(D22-K): track 28.6 -> 28.1 mm
- net Net-(D21-K): track 14.7 -> 14.2 mm
- net GND: vias 63 -> 67
Other:
- board size 243 x 27 mm -> 243 x 25 mm
